Commit message: feat: add forward kinematics (FK.py)

File: mjcf/x5_2025.urdf (robot description, URDF)
Before this commit: robot ultron_v1.1_aa, 7 links, 6 joints
Links:
- link base_link: geometry collision mesh filename=../assets/meshes/base_link.STL; visual mesh filename=../assets/meshes/base_link.STL
- link link1: geometry collision mesh filename=../assets/meshes/link1.STL; visual mesh filename=../assets/meshes/link1.STL
- link link2: geometry collision mesh filename=../assets/meshes/link2.STL; visual mesh filename=../assets/meshes/link2.STL
- link link3: geometry collision mesh filename=../assets/meshes/link3.STL; visual mesh filename=../assets/meshes/link3.STL
- link link4: geometry collision mesh filename=../assets/meshes/link4.STL; visual mesh filename=../assets/meshes/link4.STL
- link link5: geometry collision mesh filename=../assets/meshes/link5.STL; visual mesh filename=../assets/meshes/link5.STL
- link link6: geometry collision mesh filename=../assets/meshes/link6.STL; visual mesh filename=../assets/meshes/link6.STL
